Commit message: change global planner try template_matching

File: src/jackal_description/urdf/accessories.urdf.xacro (robot description, xacro)
@@ -269,5 +269,5 @@
     <xacro:pointgrey_flea3 frame="${prefix}_camera" name="${name}"
       camera_x="0.0754" camera_y="0.029" camera_z="0.029"
-      camera_mass="0.085" hfov="1.0471975512" fps="60" width="640" height="512"/>
+      camera_mass="0.05" hfov="1.0471975512" fps="60" width="640" height="512"/>
     <!-- Mount Enabled -->
     <xacro:if value="${tower}">
@@ -280,5 +280,5 @@
       </joint>
       <joint name="${prefix}_camera_bracket_joint" type="fixed">
-        <origin xyz="0.020 0 0.0245" rpy="0 0 0" />
+        <origin xyz="0.020 0 5" rpy="0 1.570795 0" />
         <parent link="${prefix}_camera_beam" />
         <child link="${prefix}_camera" />

Commit message: teb+d435

File: src/jackal_description/urdf/accessories.urdf.xacro (robot description, xacro)
@@ -256,4 +256,11 @@
     - JACKAL_BB2
   -->
+    <!-- d435 -->
+  <xacro:include filename="$(find jackal_description)/urdf/gazebo/d435.urdf.xacro" />
+  <xacro:if value="$(optenv intel_realsense 1)">
+    <xacro:sensor_d435 name="camera_front" topics_ns="camera_front" parent="base_link">
+      <origin xyz="0.2 0.0 0.184" rpy="0.0 0.0 0.0"/>
+    </xacro:sensor_d435>
+  </xacro:if>
   <!-- Common camera mounts and accessory URDFs. -->
   <xacro:include filename="$(find jackal_description)/urdf/accessories/camera_mount.urdf.xacro" />
@@ -269,5 +276,5 @@
     <xacro:pointgrey_flea3 frame="${prefix}_camera" name="${name}"
       camera_x="0.0754" camera_y="0.029" camera_z="0.029"
-      camera_mass="0.085" hfov="1.0471975512" fps="60" width="640" height="512"/>
+      camera_mass="0.05" hfov="1.0471975512" fps="60" width="640" height="512"/>
     <!-- Mount Enabled -->
     <xacro:if value="${tower}">
@@ -280,5 +287,5 @@
       </joint>
       <joint name="${prefix}_camera_bracket_joint" type="fixed">
-        <origin xyz="0.020 0 0.0245" rpy="0 0 0" />
+        <origin xyz="0.020 0 5" rpy="0 1.570795 0" />
         <parent link="${prefix}_camera_beam" />
         <child link="${prefix}_camera" />

Commit message: 修改了d435位置

File: src/jackal_description/urdf/accessories.urdf.xacro (robot description, xacro)
@@ -262,5 +262,5 @@
   <xacro:if value="$(optenv intel_realsense 1)">
     <xacro:sensor_d435 name="camera_front" topics_ns="camera_front" parent="base_link">
-      <origin xyz="0.12 0.0 0.184" rpy="0.0 0.0 0.0"/>
+      <origin xyz="0.2 0.1 0.184" rpy="0.0 0.0 0.0"/>
     </xacro:sensor_d435>
   </xacro:if>

Commit message: add detection

File: src/jackal_description/urdf/accessories.urdf.xacro (robot description, xacro)
@@ -287,5 +287,5 @@
       </joint>
       <joint name="${prefix}_camera_bracket_joint" type="fixed">
-        <origin xyz="0.020 0 5" rpy="0 1.570795 0" />
+        <origin xyz="3.020 0 10" rpy="0 1.570795 0" />
         <parent link="${prefix}_camera_beam" />
         <child link="${prefix}_camera" />
